File: hardware/KiCAD/ProPrj_CAN_2025-04-09.kicad_pcb (KiCad board)
At the start: 2 copper layers, 27.8 x 40.4 mm, 20 parts

Commit message: edit
Parts:
- removed ?: , ProPrj_CAN_2025-04-09:Pad_ie6
- removed ?: , ProPrj_CAN_2025-04-09:Pad_ie7
- removed ?: , ProPrj_CAN_2025-04-09:Pad_ie5
- removed ?: , ProPrj_CAN_2025-04-09:Pad_ie8
- removed P1: , ProPrj_CAN_2025-04-09:HDR1X7
- removed P2, P3: , ProPrj_CAN_2025-04-09:HDR1X2
- removed P4: , ProPrj_CAN_2025-04-09:TERMINAL-BLOCK-2-PIN-3.5MM-ROUND-PAD
- removed POW: , ProPrj_CAN_2025-04-09:CHIPLED_0603
- removed X1: , ProPrj_CAN_2025-04-09:HC-49US_L11.5-W4.5-P4.88
- added C6: 22 pF, Capacitor_SMD:C_0603_1608Metric_Pad1.08x0.95mm_HandSolder, F.Cu at (164.6, 123.3)
- added C7: 22 pF, Capacitor_SMD:C_0603_1608Metric_Pad1.08x0.95mm_HandSolder, F.Cu at (184.9, 118.3)
- added CRYSTAL-ECS-100-?-?PVX1: 8MHz, ProPrj_CAN_2025-04-09:HC-49US_L11.5-W4.5-P4.88, F.Cu at (190.0, 123.6)
- added D1: SS510C, Diode_SMD:D_SMB-SMC_Universal_Handsoldering, F.Cu at (192.6, 86.3)
- added D2: SS510C, Diode_SMD:D_SMB-SMC_Universal_Handsoldering, F.Cu at (192.6, 94.1)
- added D3: SMAJ33CA, Diode_SMD:D_SMA, F.Cu at (202.8, 91.3)
- added L1: 100 uH, Inductor_SMD:L_12x12mm_H8mm, F.Cu at (191.9, 106.8)
- added L2: BLM18PG121SN1D, Inductor_SMD:L_0201_0603Metric_Pad0.64x0.40mm_HandSolder, F.Cu at (202.6, 96.7)
- added MCP2: MCP2515-I, ProPrj_CAN_2025-04-09:SOIC-18_L11.6-W7.5-P1.27-LS10.3-BL, F.Cu at (173.0, 116.6)
- added U3: TJA1050DRG, ProPrj_CAN_2025-04-09:SOIC-8E, F.Cu at (203.0, 85.9)
- added U4: ESP-12F, RF_Module:ESP-12E, F.Cu at (173.2, 94.8)
- C1: value (none) -> 470 uF; footprint ProPrj_CAN_2025-04-09:tantalum A -> Capacitor_SMD:C_Elec_8x10.2
- C2, C3, C5: value (none) -> 100 nF; footprint ProPrj_CAN_2025-04-09:C0603 -> Capacitor_SMD:C_0603_1608Metric_Pad1.08x0.95mm_HandSolder
- C4: value (none) -> 470 uF; footprint ProPrj_CAN_2025-04-09:C0603 -> Capacitor_SMD:C_Elec_8x10.2
- R1, R2, R3: value (none) -> 10 k; footprint ProPrj_CAN_2025-04-09:R0603 -> Resistor_SMD:R_0603_1608Metric_Pad0.98x0.95mm_HandSolder
- U1: value (none) -> LM2575-5.0BT; footprint ProPrj_CAN_2025-04-09:SOIC-8E -> Package_TO_SOT_SMD:TO-263-5_TabPin3
- U2: value (none) -> AMS1117-3.3; footprint ProPrj_CAN_2025-04-09:SOIC-18_L11.6-W7.5-P1.27-LS10.3-BL -> Package_TO_SOT_SMD:SOT-223-3_TabPin2
- moved R1 69.6 mm to (200.9, 109.9)
- moved R3 22.9 mm to (161.4, 99.6)
- moved C5 20.7 mm to (158.5, 103.5)
- moved U2 19.4 mm to (157.1, 87.0)
- moved C1 16.6 mm to (144.8, 86.7), turned to 90 degrees
- moved C3 9.70 mm to (157.1, 116.0)
- moved R2 9.70 mm to (141.9, 113.9)
- moved C4 7.58 mm to (157.1, 112.3)
- moved U1 5.83 mm to (143.5, 111.9)
- moved C2 4.30 mm to (140.8, 99.5), turned to 180 degrees
Connections:
- C1 pad 1: (no net) -> VCC
- C1 pad 2: (no net) -> GND
- C2 pad 1: (no net) -> VCC
- C2 pad 2: (no net) -> GND
- C3 pad 1: (no net) -> VCC
- C3 pad 2: (no net) -> GND
- C4 pad 1: (no net) -> Net-(D2-K)
- C4 pad 2: (no net) -> GND
- C5 pad 1: (no net) -> Net-(D2-K)
- C5 pad 2: (no net) -> GND
- R1 pad 1: (no net) -> VCC
- R1 pad 2: (no net) -> Net-(MCP2-~RESET~)
- R2 pad 1: (no net) -> Net-(J1-Pin_1)
- R2 pad 2: (no net) -> Net-(U3-CANH)
- R3 pad 1: (no net) -> +3.3V
- R3 pad 2: (no net) -> Net-(U4-EN)
- U1 pad 1: (no net) -> Net-(D2-K)
- U1 pad 2: (no net) -> Net-(D1-K)
- U1 pad 3: (no net) -> GND
- U1 pad 4: (no net) -> VCC
- U1 pad 5: (no net) -> GND
- U2 pad 1: (no net) -> GND
- U2 pad 2: (no net) -> +3.3V
- U2 pad 3: (no net) -> VCC
Routing:
- net 0: track 160.7 -> 0.00 mm, vias 6 -> 0
- removed copper zone on B.Cu, net (none)
- removed copper zone on F.Cu, net (none)
Other:
- board size 27.8 x 40.4 mm -> 85.2 x 50.9 mm
- board text removed: "CAN Bus Module"
- board text removed: "CS"
- board text removed: "GND"
- board text removed: "INT"
- board text removed: "L"
- board text removed: "SCK"
- board text removed: "SI"
- board text removed: "SO"
- board text removed: "VCC"

Commit message: reorder
Parts:
- added F1: MF-SM185/33-2, Inductor_SMD:L_0603_1608Metric_Pad1.05x0.95mm_HandSolder, F.Cu at (212.6, 111.9)
- added J1: KF2510-4, Connector_Molex:Molex_KK-254_AE-6410-04A_1x04_P2.54mm_Vertical, F.Cu at (211.7, 99.8)
- added J3: RESET, Connector_PinSocket_2.54mm:PinSocket_1x02_P2.54mm_Vertical, F.Cu at (182.5, 82.7)
- added J4: PROG, Connector_PinHeader_2.54mm:PinHeader_1x04_P2.54mm_Vertical, F.Cu at (175.4, 82.3)
- added J5: BOOT, Connector_PinSocket_2.54mm:PinSocket_1x02_P2.54mm_Vertical, F.Cu at (175.4, 100.8)
- added R4: 10 k, Resistor_SMD:R_0603_1608Metric_Pad0.98x0.95mm_HandSolder, F.Cu at (178.8, 83.8)
- added Y1: Crystal, Crystal:Crystal_SMD_HC49-SD_HandSoldering, F.Cu at (204.2, 81.8)
- L1: footprint Inductor_SMD:L_12x12mm_H8mm -> Inductor_SMD:L_SXN_SMDRI127
- L2: footprint Inductor_SMD:L_0201_0603Metric_Pad0.64x0.40mm_HandSolder -> Inductor_SMD:L_0603_1608Metric_Pad1.05x0.95mm_HandSolder
- R2: value 10 k -> 120
- moved R2 66.9 mm to (205.8, 94.1), turned to 90 degrees
- moved C6 51.0 mm to (201.0, 87.6), turned to -90 degrees
- moved C5 49.8 mm to (206.8, 115.6), turned to 90 degrees
- moved C1 48.4 mm to (189.8, 104.4), turned to -90 degrees
- moved U1 45.2 mm to (187.5, 122.6)
- moved CRYSTAL-ECS-100-?-?PVX1 44.3 mm to (204.3, 81.7)
- moved C4 43.3 mm to (200.4, 112.2), turned to 90 degrees
- moved C7 36.8 mm to (205.4, 87.6), turned to 90 degrees
- moved D2 33.1 mm to (208.0, 123.3)
- moved MCP2 32.1 mm to (192.0, 90.7), turned to 90 degrees
- moved U2 32.0 mm to (156.7, 119.0)
- moved D1 28.7 mm to (175.8, 109.6)
- moved C2 28.0 mm to (167.4, 108.2), turned to 90 degrees
- moved C3 27.2 mm to (180.4, 101.9), turned to 90 degrees
- moved L1 25.9 mm to (170.8, 121.8), turned to 180 degrees
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Other:
- board size 85.2 x 50.9 mm -> 66.2 x 50.9 mm
- board text removed: "H"
