File: hardware/KiCAD/ProPrj_CAN_2025-04-09.kicad_pcb (KiCad board)
At the start: 2 copper layers, 66.2 x 50.9 mm, 28 parts, among them J1 KF2510-4, J3 RESET, J4 PROG, J5 BOOT, U1 LM2575-5.0BT, U2 AMS1117-3.3, U3 TJA1050DRG, U4 ESP-12F, Y1 Crystal

Commit message: reorder
Parts:
- removed the J3 at (182.5, 82.7)
- removed J4: PROG, Connector_PinHeader_2.54mm:PinHeader_1x04_P2.54mm_Vertical
- removed J5: BOOT, Connector_PinSocket_2.54mm:PinSocket_1x02_P2.54mm_Vertical
- added J1: BOOT, Connector_PinHeader_2.54mm:PinHeader_1x03_P2.54mm_Vertical, F.Cu at (180.3, 83.1)
- added J2: PROG, Connector_PinHeader_2.54mm:PinHeader_1x03_P2.54mm_Vertical, F.Cu at (176.7, 83.1)
- moved R2 28.1 mm to (151.5, 90.6)
- renumbered C5 to C2, C4 to C3, C2 to C4, C7 to C5, C3 to C7, D3 to D1, D1 to D3, J1 to J3, L2 to L1, L1 to L2, R4 to R2, R2 to R4, MCP2 to U2, U2 to U3, U3 to U4, U4 to U5
Routing:
- net GND: track 0.00 -> 212.4 mm, vias 0 -> 15
- net VCC: track 0.00 -> 118.7 mm
- net +3.3V: track 0.00 -> 68.7 mm
- net Net-(U2-SI): track 0.00 -> 39.6 mm
- net Net-(D3-K): track 0.00 -> 36.8 mm
- net Net-(U2-SCK): track 0.00 -> 34.7 mm
- net Net-(U2-SO): track 0.00 -> 34.5 mm
- net Net-(D2-K): track 0.00 -> 24.2 mm
- net Net-(U2-RXCAN): track 0.00 -> 21.4 mm, vias 0 -> 2
- net Net-(U2-OSC2): track 0.00 -> 20.6 mm
- net Net-(U2-~CS~): track 0.00 -> 19.6 mm
- net Net-(J1-Pin_2): track 0.00 -> 18.8 mm, vias 0 -> 1
- net Net-(U2-~INT~): track 0.00 -> 18.4 mm
- net Net-(J3-Pin_2): track 0.00 -> 18.0 mm, vias 0 -> 1
- net Net-(D1-A2): track 0.00 -> 14.4 mm
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- added copper zone on B.Cu, net GND
- added copper zone on F.Cu, net GND
Other:
- board size 66.2 x 50.9 mm -> 66 x 50 mm

Commit message: Rouring
Parts:
- removed CRYSTAL-ECS-100-?-?PVX1: 8MHz, ProPrj_CAN_2025-04-09:HC-49US_L11.5-W4.5-P4.88
- added C8: 470 uF, Capacitor_SMD:C_Elec_8x10.2, F.Cu at (106.6, 82.8)
- added C9: 100 nF, Capacitor_SMD:C_0603_1608Metric_Pad1.08x0.95mm_HandSolder, F.Cu at (104.4, 71.8)
- F1: footprint Inductor_SMD:L_0603_1608Metric_Pad1.05x0.95mm_HandSolder -> Library:FUSE_MF-SM185_BRN
- L1: value BLM18PG121SN1D -> BLM21PG300SN1D; footprint Inductor_SMD:L_0603_1608Metric_Pad1.05x0.95mm_HandSolder -> Inductor_SMD:L_0805_2012Metric_Pad1.05x1.20mm_HandSolder
- Y1: value Crystal -> 8 - 16 MHz; footprint Crystal:Crystal_SMD_HC49-SD_HandSoldering -> Library:Crystal_SMD_HC49-SD_HandSoldering
- moved C2 71.8 mm to (143.3, 82.2)
- moved C5 65.4 mm to (150.3, 52.4), turned to -90 degrees
- moved L1 65.4 mm to (150.0, 81.9), turned to -90 degrees
- moved R1 62.1 mm to (129.1, 65.3)
- moved U1 61.1 mm to (134.8, 91.8)
- moved D3 60.5 mm to (122.6, 80.8), turned to 180 degrees
- moved C7 60.5 mm to (132.2, 65.3)
- moved U2 60.4 mm to (141.4, 57.7)
- moved C6 59.6 mm to (150.3, 56.3)
- moved F1 59.5 mm to (159.3, 85.5), turned to 0 degrees
- moved C4 59.2 mm to (114.5, 81.5)
- moved L2 59.2 mm to (119.5, 92.2)
- moved C1 59.1 mm to (139.4, 73.6), turned to 90 degrees
- moved U4 59.0 mm to (162.1, 56.4), turned to -90 degrees
- moved C3 57.3 mm to (146.7, 92.3)
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Connections:
- F1 pad 1: +12V -> Net-(D1-A2)
- F1 pad 2: Net-(D1-A2) -> +12V
- R4 pad 2: Net-(U4-CANH) -> Net-(J3-Pin_2)
- U4 pad 7: Net-(U4-CANH) -> Net-(J3-Pin_1)
Routing:
- net GND: track 212.4 -> 50.8 mm, vias 15 -> 22
- net Net-(U2-TXCAN): track 13.7 -> 37.3 mm
- net Net-(U2-~CS~): track 19.6 -> 0.00 mm
- net Net-(D2-K): track 24.2 -> 41.6 mm
- net Net-(D3-K): track 36.8 -> 24.7 mm
- net Net-(U2-RXCAN): track 21.4 -> 32.5 mm, vias 2 -> 0
- net +3.3V: track 68.7 -> 78.3 mm
- net Net-(U4-CANH): track 8.24 -> 0.00 mm
- net VCC: track 118.7 -> 113.1 mm, vias 0 -> 4
- net Net-(U2-OSC2): track 20.6 -> 15.9 mm
- net Net-(J3-Pin_1): track 7.86 -> 12.4 mm
- net Net-(J1-Pin_2): track 18.8 -> 14.7 mm
- net Net-(U2-~RESET~): track 4.69 -> 8.69 mm
- net Net-(U2-SI): track 39.6 -> 36.4 mm
- net Net-(U2-SO): track 34.5 -> 31.3 mm
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- removed copper zone on F.Cu, net GND

Commit message: ok
Parts:
- moved C1 3.73 mm to (135.7, 73.3), turned to 0 degrees
- moved U3 0.21 mm to (106.2, 94.5)
Routing:
- net GND: track 50.8 -> 21.3 mm, vias 22 -> 21
- net Net-(U2-~CS~): track 0.00 -> 23.0 mm, vias 0 -> 2
- net Net-(U2-RXCAN): track 32.5 -> 16.7 mm, vias 0 -> 2
- net VCC: track 113.1 -> 98.3 mm
- net Net-(U2-TXCAN): track 37.3 -> 22.6 mm, vias 0 -> 2
- net +3.3V: track 78.3 -> 89.1 mm
- net Net-(U2-~INT~): track 19.6 -> 24.6 mm
- net Net-(U2-OSC2): track 15.9 -> 11.3 mm
- net Net-(D2-K): track 41.6 -> 37.6 mm
- net Net-(U2-SO): track 31.3 -> 34.6 mm, vias 0 -> 2
- net Net-(U2-SI): track 36.4 -> 39.2 mm, vias 0 -> 2
- net Net-(U2-SCK): track 32.7 -> 34.8 mm, vias 0 -> 2
- net Net-(J3-Pin_1): track 12.4 -> 11.0 mm
- net Net-(J1-Pin_2): vias 1 -> 0
- added copper zone on F.Cu, net GND
