File: hardware/KiCAD/ProPrj_CAN_2025-04-09.kicad_pcb (KiCad board)
At the start: 2 copper layers, 66 x 50 mm, 28 parts, among them J1 BOOT, J2 PROG, J3 KF2510-4, U1 LM2575-5.0BT, U2 MCP2515-I, U3 AMS1117-3.3, U4 TJA1050DRG, U5 ESP-12F, Y1 8 - 16 MHz

Commit message: aa
Parts:
- D1: footprint Diode_SMD:D_SMA -> Diode_SMD:D_SMB-SMC_Universal_Handsoldering
- J1: value BOOT -> PLS-3
- J2: value PROG -> PLS-3
- L2: value 100 uH -> 220 uH; footprint Inductor_SMD:L_SXN_SMDRI127 -> Library:L_12x12_universal
- U2: footprint ProPrj_CAN_2025-04-09:SOIC-18_L11.6-W7.5-P1.27-LS10.3-BL -> Library:SOIC-18_L11.6-W7.5-P1.27-LS10.3-BL
- U4: footprint ProPrj_CAN_2025-04-09:SOIC-8E -> Library:SOIC-8E
- Y1: footprint Library:Crystal_SMD_HC49-SD_HandSoldering -> Library:Crystal_SMD_THT_HC49_HandSoldering
- moved L1 7.85 mm to (155.0, 75.8)
- moved D1 5.82 mm to (148.5, 76.8)
- moved J3 1.80 mm to (160.5, 71.2)
- moved Y1 0.34 mm to (154.5, 60.8)
Routing:
- net Net-(D2-A): track 13.1 -> 20.6 mm
- net Net-(D1-A2): track 12.5 -> 17.6 mm
- net GND: track 21.3 -> 26.1 mm, vias 21 -> 42
- net Net-(J3-Pin_1): track 11.0 -> 12.8 mm
- net Net-(U2-SCK): track 34.8 -> 36.6 mm
- net Net-(U2-SO): track 34.6 -> 36.3 mm
- net Net-(J3-Pin_2): track 15.6 -> 17.1 mm
- net +12V: track 6.78 -> 7.71 mm
- net Net-(J1-Pin_2): track 14.7 -> 13.8 mm
- net Net-(U2-SI): track 39.2 -> 38.5 mm
- net +3.3V: track 89.1 -> 89.6 mm
Other:
- board text added: "+"
- board text added: "3.3V"
- board text added: "GND"
- board text added: "H"
- board text added: "L"
- board text added: "RX/TX"
- board text added: "⊥"
