File: hardware/KiCAD/ProPrj_CAN_2025-04-09.kicad_sch (KiCad schematic)
At the start: 18 parts, among them J1 Conn_01x04_Pin, U1 TJA1050DRG, U2 MCP2515-I, U3 ESP-12F, U4 LM2575HVR-5.0, U5 AMS1117-3.3, X1 8MHz

Commit message: edit
Parts:
- removed C1: 10uF/16V, ProPrj_CAN-easyedapro:tantalum A, symbol ProPrj_CAN-easyedapro:Cap_Tantalum
- removed C2, C5: 100nF, ProPrj_CAN-easyedapro:C0603, symbol ProPrj_CAN-easyedapro:Cap_0603
- removed C3, C4: 22pF, ProPrj_CAN-easyedapro:C0603, symbol ProPrj_CAN-easyedapro:Cap_0603
- removed LEDCHIP-LED0603: RED LED, ProPrj_CAN-easyedapro:CHIPLED_0603, symbol ProPrj_CAN-easyedapro:LEDCHIP-LED0603
- removed R1: 1kΩ, ProPrj_CAN-easyedapro:R0603, symbol ProPrj_CAN-easyedapro:Res_0603
- removed R2: 120Ω, ProPrj_CAN-easyedapro:R0603, symbol ProPrj_CAN-easyedapro:Res_0603
- removed R3: 10kΩ, ProPrj_CAN-easyedapro:R0603, symbol ProPrj_CAN-easyedapro:Res_0603
- removed U2: MCP2515-I, ProPrj_CAN-easyedapro:SOIC-18_L11.6-W7.5-P1.27-LS10.3-BL, symbol ProPrj_CAN-easyedapro:MCP2515
- added C1, C4: 470 uF, Capacitor_SMD:C_Elec_8x10.2, symbol Device:C_Polarized
- added C2, C3, C5: 100 nF, Capacitor_SMD:C_0603_1608Metric_Pad1.08x0.95mm_HandSolder, symbol Device:C
- added C6, C7: 22 pF, Capacitor_SMD:C_0603_1608Metric_Pad1.08x0.95mm_HandSolder, symbol Device:C
- added D2: SS510C, Diode_SMD:D_SMB-SMC_Universal_Handsoldering, symbol Device:D_Schottky
- added D3: SMAJ33CA, Diode_SMD:D_SMA, symbol Diode:SMAJ33CA
- added F1: MF-SM185/33-2, symbol Device:Polyfuse
- added J2: Programm, symbol Connector_Generic:Conn_01x04
- added J3: BOOT, symbol Connector_Generic:Conn_01x02
- added J4: RESET, symbol Connector_Generic:Conn_01x02
- added L2: BLM18PG121SN1D, Inductor_SMD:L_0201_0603Metric_Pad0.64x0.40mm_HandSolder, symbol Device:L_Ferrite
- added MCP2: MCP2515-I, ProPrj_CAN_2025-04-09:SOIC-18_L11.6-W7.5-P1.27-LS10.3-BL, symbol ProPrj_CAN-easyedapro:MCP2515-I-01
- added R1, R2, R3: 10 k, Resistor_SMD:R_0603_1608Metric_Pad0.98x0.95mm_HandSolder, symbol Device:R
- CRYSTAL-ECS-100-?-?PVX1: renamed from X1; footprint ProPrj_CAN-easyedapro:HC-49US_L11.5-W4.5-P4.88 -> ProPrj_CAN_2025-04-09:HC-49US_L11.5-W4.5-P4.88
- D1: value B540C-13-F -> SS510C; footprint (none) -> Diode_SMD:D_SMB-SMC_Universal_Handsoldering
- J1: value Conn_01x04_Pin -> KF2510-4
- L1: value 220 uH -> 100 uH; footprint (none) -> Inductor_SMD:L_12x12mm_H8mm
- U1: renamed from U4; value LM2575HVR-5.0 -> LM2575-5.0BT; footprint Package_TO_SOT_THT:TO-220-5_Vertical -> Package_TO_SOT_SMD:TO-263-5_TabPin3
- U3: renamed from U1; footprint ProPrj_CAN-easyedapro:SOIC-8E -> ProPrj_CAN_2025-04-09:SOIC-8E
- renumbered U5 to U2, U3 to U4
Connections:
- net GND: now also C1.2, C2.2, C3.2, C4.2, C5.2, C6.1, C7.1, D3.1 (A1), J2.1 (Pin_1), J3.1 (Pin_1), J4.1 (Pin_1), MCP2.9 (VSS)
- net VCC: now also C1.1, C2.1, C3.1, MCP2.18 (VDD), R1.1
- net at J1.1 (Pin_1): now also R2.1
- net at U3.7 (CANH): now also R2.2
- net at U3.1 (TXD): now also MCP2.1 (TXCAN)
- net at U4.20 (GPIO5): now also MCP2.12 (~INT~)
- net at U4.5 (GPIO14): now also MCP2.13 (SCK)
- net at U4.7 (GPIO13): now also MCP2.14 (SI)
- net at U4.6 (GPIO12): now also MCP2.15 (SO)
- net at U4.16 (GPIO15): now also MCP2.16 (~CS~)
- net at U3.4 (RXD): now also MCP2.2 (RXCAN)
- net at CRYSTAL-ECS-100-?-?PVX1.2: now also C6.2, MCP2.7 (OSC2)
- net at CRYSTAL-ECS-100-?-?PVX1.1: now also C7.2, MCP2.8 (OSC1)
- net at U4.1 (~{RST}): now also J4.2 (Pin_2)
- net at U4.18 (GPIO0): now also J3.2 (Pin_2)
- net at U4.21 (GPIO3/RXD): now also J2.3 (Pin_3)
- net at U4.22 (GPIO1/TXD): now also J2.2 (Pin_2)
- net at U4.3 (EN): now also R3.2
- net Board_PWR 12V: no longer names the net of U1.1 (VIN)
- net Board_PWR 12V: now also C4.1, C5.1, D2.1 (K); no longer J1.4 (Pin_4)
- net VCC 3.3 V renamed +3.3V
- net +3.3V: now also J2.4 (Pin_4), R3.1
- new net: MCP2.17 (~RESET~), R1.2
- new net: D3.2 (A2), F1.2, L2.1
- new net: D2.2 (A), L2.2
- new net +12V: F1.1, J1.4 (Pin_4)
- no-connect marks 0 -> 16
Other:
- note removed: "100nF"
- note removed: "10K"
- note removed: "10uF/16V"
- note removed: "120R"
- note removed: "1K"
- note removed: "22pF"
- moved on the sheet: J1

Commit message: reorder
Parts:
- removed J2: Programm, symbol Connector_Generic:Conn_01x04
- removed J3: BOOT, symbol Connector_Generic:Conn_01x02
- removed J4: RESET, symbol Connector_Generic:Conn_01x02
- added J3: RESET, Connector_PinSocket_2.54mm:PinSocket_1x02_P2.54mm_Vertical, symbol Connector:Conn_01x02_Pin
- added J4: PROG, Connector_PinHeader_2.54mm:PinHeader_1x04_P2.54mm_Vertical, symbol Connector:Conn_01x04_Pin
- added J5: BOOT, Connector_PinSocket_2.54mm:PinSocket_1x02_P2.54mm_Vertical, symbol Connector:Conn_01x02_Pin
- added R4: 10 k, Resistor_SMD:R_0603_1608Metric_Pad0.98x0.95mm_HandSolder, symbol Device:R
- added Y1: Crystal, Crystal:Crystal_SMD_HC49-SD_HandSoldering, symbol Device:Crystal
- F1: footprint (none) -> Inductor_SMD:L_0603_1608Metric_Pad1.05x0.95mm_HandSolder
- J1: footprint (none) -> Connector_Molex:Molex_KK-254_AE-6410-04A_1x04_P2.54mm_Vertical
- L1: footprint Inductor_SMD:L_12x12mm_H8mm -> Inductor_SMD:L_SXN_SMDRI127
- L2: footprint Inductor_SMD:L_0201_0603Metric_Pad0.64x0.40mm_HandSolder -> Inductor_SMD:L_0603_1608Metric_Pad1.05x0.95mm_HandSolder
- R2: value 10 k -> 120
Connections:
- net +3.3V: now also J4.4 (Pin_4), R4.1
- net GND: now also J3.1 (Pin_1), J4.1 (Pin_1), J5.1 (Pin_1)
- net at C6.2, CRYSTAL-ECS-100-?-?PVX1.2, MCP2.7 (OSC2): now also Y1.2
- net at U4.18 (GPIO0): now also J5.2 (Pin_2)
- net at C7.2, CRYSTAL-ECS-100-?-?PVX1.1, MCP2.8 (OSC1): now also Y1.1
- net at U4.1 (~{RST}): now also J3.2 (Pin_2), R4.2
- net at U4.21 (GPIO3/RXD): now also J4.3 (Pin_3)
- net at U4.22 (GPIO1/TXD): now also J4.2 (Pin_2)
Other:
- moved on the sheet: C6, C7, CRYSTAL-ECS-100-?-?PVX1, R3

Commit message: reorder
Parts:
- removed J3: RESET, Connector_PinSocket_2.54mm:PinSocket_1x02_P2.54mm_Vertical, symbol Connector:Conn_01x02_Pin
- removed J4: PROG, Connector_PinHeader_2.54mm:PinHeader_1x04_P2.54mm_Vertical, symbol Connector:Conn_01x04_Pin
- removed J5: BOOT, Connector_PinSocket_2.54mm:PinSocket_1x02_P2.54mm_Vertical, symbol Connector:Conn_01x02_Pin
- added J1: BOOT, Connector_PinHeader_2.54mm:PinHeader_1x03_P2.54mm_Vertical, symbol Connector:Conn_01x03_Pin
- added J2: PROG, Connector_PinHeader_2.54mm:PinHeader_1x03_P2.54mm_Vertical, symbol Connector:Conn_01x03_Pin
- renumbered C5 to C2, C4 to C3, C2 to C4, C7 to C5, C3 to C7, D3 to D1, D1 to D3, J1 to J3, L2 to L1, L1 to L2, R4 to R2, R2 to R4, MCP2 to U2, U2 to U3, U3 to U4, U4 to U5
Connections:
- net +3.3V: now also J1.3 (Pin_3)
- net GND: now also J1.1 (Pin_1), J2.1 (Pin_1)
- net at U5.22 (GPIO1/TXD): now also J2.2 (Pin_2)
- net at U5.21 (GPIO3/RXD): now also J2.3 (Pin_3)
- net at U5.18 (GPIO0): now also J1.2 (Pin_2)
Other:
- moved on the sheet: R2

Commit message: Rouring
Parts:
- removed CRYSTAL-ECS-100-?-?PVX1: 8MHz, ProPrj_CAN_2025-04-09:HC-49US_L11.5-W4.5-P4.88, symbol ProPrj_CAN-easyedapro:CRYSTAL-ECS-100-20-5PVX
- added C8: 470 uF, Capacitor_SMD:C_Elec_8x10.2, symbol Device:C_Polarized
- added C9: 100 nF, Capacitor_SMD:C_0603_1608Metric_Pad1.08x0.95mm_HandSolder, symbol Device:C
- F1: footprint Inductor_SMD:L_0603_1608Metric_Pad1.05x0.95mm_HandSolder -> Library:FUSE_MF-SM185_BRN; symbol Device:Polyfuse -> Local:MF-SM185_33-2
- L1: value BLM18PG121SN1D -> BLM21PG300SN1D; footprint Inductor_SMD:L_0603_1608Metric_Pad1.05x0.95mm_HandSolder -> Inductor_SMD:L_0805_2012Metric_Pad1.05x1.20mm_HandSolder
- Y1: value Crystal -> 8 - 16 MHz; footprint Crystal:Crystal_SMD_HC49-SD_HandSoldering -> Library:Crystal_SMD_HC49-SD_HandSoldering
Connections:
- net +12V: now also F1.2; no longer F1.1
- net +3.3V: now also C8.1, C9.1
- net GND: now also C8.2, C9.2
- net at D1.2 (A2), L1.1: now also F1.1; no longer F1.2
- net at J3.1 (Pin_1), R4.1: now also U4.7 (CANH)
- net at J3.2 (Pin_2), U4.6 (CANL): now also R4.2
Other:
- note removed: "8MHz"

Commit message: aa
Parts:
- C1, C3, C8: value 470 uF -> 100 uF 50V; ChipDip (none) -> 9000364655
- C2, C4, C7, C9: ChipDip (none) -> 9000121254
- C5, C6: ChipDip (none) -> 183744283
- D1: footprint Diode_SMD:D_SMA -> Diode_SMD:D_SMB-SMC_Universal_Handsoldering; ChipDip (none) -> 9001169250
- D2, D3: ChipDip (none) -> 9001106124
- F1: ChipDip (none) -> 9000451773
- J1: value BOOT -> PLS-3; ChipDip (none) -> 132511368
- J2: value PROG -> PLS-3; ChipDip (none) -> 132511368
- J3: ChipDip (none) -> 8014106147
- L1: ChipDip (none) -> 9000180593
- L2: value 100 uH -> 220 uH; footprint Inductor_SMD:L_SXN_SMDRI127 -> Library:L_12x12_universal; ChipDip (none) -> 970844433
- R1, R2, R3: ChipDip (none) -> 9000079736
- R4: ChipDip (none) -> 9000079618
- U1: symbol Regulator_Switching:LM2575-5.0BT -> Local:LM2575-5.0BT; ChipDip (none) -> 9001087019
- U2: footprint ProPrj_CAN_2025-04-09:SOIC-18_L11.6-W7.5-P1.27-LS10.3-BL -> Library:SOIC-18_L11.6-W7.5-P1.27-LS10.3-BL; ChipDip (none) -> 2534353951
- U3: symbol Regulator_Linear:AMS1117-3.3 -> Local:AMS1117-3.3; ChipDip (none) -> 9020004445
- U4: footprint ProPrj_CAN_2025-04-09:SOIC-8E -> Library:SOIC-8E; symbol ProPrj_CAN-easyedapro:TJA1050DRG -> Local:TJA1050DRG; ChipDip (none) -> 8044731834
- U5: symbol RF_Module:ESP-12F -> Local:ESP-12F; ChipDip (none) -> 8009379123
- Y1: footprint Library:Crystal_SMD_HC49-SD_HandSoldering -> Library:Crystal_SMD_THT_HC49_HandSoldering; symbol Device:Crystal -> Local:Crystal; ChipDip (none) -> 9001626980
Changed lines of the file:
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@@
 			)
 		)
-		(property "Value" "470 uF"
+		(property "Value" "100 uF 50V"
 			(at 178.816 145.542 0)
 			(effects
@@
 			)
 		)
-		(property "Datasheet" "https://static.chipdip.ru/lib/074/DOC012074579.pdf"
+		(property "Datasheet" "https://www.chipdip.ru/product/eeefk1h101p"
 			(at 189.23 147.32 0)
 			(effects
@@
 			)
 		)
-		(property "ChipDip" ""
+		(property "ChipDip" "9000364655"
 			(at 189.23 147.32 0)
 			(effects
@@
 			)
 		)
-		(property "Datasheet" "~"
+		(property "Datasheet" "https://static.chipdip.ru/lib/538/DOC012538954.pdf"
 			(at 68.58 91.44 0)
 			(effects
@@
 			)
 		)
-		(property "ChipDip" ""
+		(property "ChipDip" "183744283"
 			(at 68.58 91.44 0)
 			(effects
@@
 			)
 		)
-		(property "Value" "100 uH"
+		(property "Value" "220 uH"
 			(at 106.68 129.54 90)
 			(effects
@@
 			)
 		)
-		(property "Footprint" "Inductor_SMD:L_SXN_SMDRI127"
+		(property "Footprint" "Library:L_12x12_universal"
 			(at 106.68 133.35 0)
 			(effects
@@
 			)
 		)
-		(property "ChipDip" ""
+		(property "ChipDip" "970844433"
 			(at 106.68 133.35 0)
 			(effects
@@
 			)
 		)
-		(property "Datasheet" "~"
+		(property "Datasheet" "https://static.chipdip.ru/lib/295/DOC021295017.pdf"
 			(at 97.79 139.7 0)
 			(effects
@@
 			)
 		)
-		(property "ChipDip" ""
+		(property "ChipDip" "9001106124"
 			(at 97.79 139.7 0)
 			(effects
@@
 	)
 	(symbol
-		(lib_id "Device:Crystal")
+		(lib_id "Local:Crystal")
 		(at 77.47 96.52 90)
 		(unit 1)
@@
 			)
 		)
-		(property "Footprint" "Library:Crystal_SMD_HC49-SD_HandSoldering"
+		(property "Footprint" "Library:Crystal_SMD_THT_HC49_HandSoldering"
 			(at 77.47 96.52 0)
 			(effects
@@
 			)
 		)
-		(property "ChipDip" ""
+		(property "ChipDip" "9001626980"
 			(at 77.47 96.52 0)
 			(effects
@@
 			)
 		)
-		(property "Datasheet" "~"
+		(property "Datasheet" "https://www.chipdip.ru/product/grm188r72a104ka35d"
 			(at 62.23 85.09 0)
 			(effects
@@
 			)
 		)
-		(property "ChipDip" ""
+		(property "ChipDip" "9000121254"
 			(at 62.23 85.09 0)
 			(effects
@@
 			)
 		)
-		(property "Datasheet" "~"
+		(property "Datasheet" "https://www.chipdip.ru/product/grm188r72a104ka35d"
 			(at 77.47 53.34 0)
 			(effects
@@
 			)
 		)
-		(property "ChipDip" ""
+		(property "ChipDip" "9000121254"
 			(at 77.47 53.34 0)
 			(effects
@@
 			)
 		)
-		(property "Datasheet" "~"
+		(property "Datasheet" "https://static.chipdip.ru/lib/175/DOC011175144.pdf"
 			(at 77.47 78.74 0)
 			(effects
@@
 			)
 		)
-		(property "ChipDip" ""
+		(property "ChipDip" "9000079736"
 			(at 77.47 78.74 0)
 			(effects
@@
 		(fields_autoplaced yes)
 		(property "Reference" "U2"
-			(at 105.41 55.88 0)
+			(at 105.41 54.61 0)
 			(effects
 				(font
@@
 			)
 		)
-		(property "Footprint" "ProPrj_CAN_2025-04-09:SOIC-18_L11.6-W7.5-P1.27-LS10.3-BL"
+		(property "Footprint" "Library:SOIC-18_L11.6-W7.5-P1.27-LS10.3-BL"
 			(at 91.44 60.96 0)
 			(effects
@@
 			)
 		)
-		(property "ChipDip" ""
+		(property "ChipDip" "2534353951"
 			(at 91.44 60.96 0)
 			(effects
@@
 			)
 		)
-		(property "Value" "470 uF"
+		(property "Value" "100 uF 50V"
 			(at 25.146 83.312 0)
 			(effects
@@
 			)
 		)
-		(property "Datasheet" "https://static.chipdip.ru/lib/074/DOC012074579.pdf"
+		(property "Datasheet" "https://www.chipdip.ru/product/eeefk1h101p"
 			(at 35.56 85.09 0)
 			(effects
@@
 			)
 		)
-		(property "ChipDip" ""
+		(property "ChipDip" "9000364655"
 			(at 35.56 85.09 0)
 			(effects
@@
 			)
 		)
-		(property "ChipDip" ""
+		(property "ChipDip" "9000451773"
 			(at 17.78 128.27 0)
 			(effects
@@
 	)
 	(symbol
-		(lib_id "RF_Module:ESP-12F")
+		(lib_id "Local:ESP-12F")
 		(at 182.88 90.17 0)
 		(unit 1)
@@
 			)
 		)
-		(property "ChipDip" ""
+		(property "ChipDip" "8009379123"
 			(at 182.88 90.17 0)
 			(effects
@@
 			)
 		)
-		(property "Datasheet" "~"
+		(property "Datasheet" "https://static.chipdip.ru/lib/629/DOC041629679.pdf"
 			(at 260.35 77.47 0)
 			(effects
@@
 			)
 		)
-		(property "ChipDip" ""
+		(property "ChipDip" "8014106147"
 			(at 260.35 77.47 0)
 			(effects
@@
 			)
 		)
-		(property "Datasheet" "~"
+		(property "Datasheet" "https://static.chipdip.ru/lib/175/DOC011175144.pdf"
 			(at 160.02 74.93 0)
 			(effects
@@
 			)
 		)
-		(property "ChipDip" ""
+		(property "ChipDip" "9000079736"
 			(at 160.02 74.93 0)
 			(effects
@@
 			)
 		)
-		(property "Value" "470 uF"
+		(property "Value" "100 uF 50V"
 			(at 61.468 141.224 0)
 			(effects
@@
 			)
 		)
-		(property "Datasheet" "https://static.chipdip.ru/lib/074/DOC012074579.pdf"
+		(property "Datasheet" "https://www.chipdip.ru/product/eeefk1h101p"
 			(at 57.15 139.7 0)
 			(effects
@@
 			)
 		)
-		(property "ChipDip" ""
+		(property "ChipDip" "9000364655"
 			(at 57.15 139.7 0)
 			(effects
@@
 			)
 		)
-		(property "Value" "PROG"
+		(property "Value" "PLS-3"
 			(at 221.234 80.264 0)
 			(effects
@@
 			)
 		)
-		(property "Datasheet" "~"
+		(property "Datasheet" "https://www.chipdip.ru/product/pls-3"
 			(at 217.17 80.01 0)
 			(effects
@@
 			)
 		)
-		(property "ChipDip" ""
+		(property "ChipDip" "132511368"
 			(at 217.17 80.01 0)
 			(effects
@@
 			)
 		)
-		(property "Datasheet" "https://www.chipdip.ru/product/blm21pg300sn1d"
+		(property "Datasheet" "https://www.chipdip.ru/product/blm21pg121sn1d"
 			(at 31.75 128.27 0)
 			(effects
@@
 			)
 		)
-		(property "ChipDip" ""
+		(property "ChipDip" "9000180593"
 			(at 31.75 128.27 0)
 			(effects
@@
 			)
 		)
-		(property "Datasheet" "~"
+		(property "Datasheet" "https://static.chipdip.ru/lib/200/DOC011200708.pdf"
 			(at 242.57 57.15 0)
 			(effects
@@
 			)
 		)
-		(property "ChipDip" ""
+		(property "ChipDip" "9000079618"
 			(at 242.57 57.15 0)
 			(effects
@@
 			)
 		)
-		(property "Datasheet" "~"
+		(property "Datasheet" "https://www.chipdip.ru/product/grm188r72a104ka35d"
 			(at 204.47 147.32 0)
 			(effects
@@
 			)
 		)
-		(property "ChipDip" ""
+		(property "ChipDip" "9000121254"
 			(at 204.47 147.32 0)
 			(effects
@@
 	)
 	(symbol
-		(lib_id "Regulator_Linear:AMS1117-3.3")
+		(lib_id "Local:AMS1117-3.3")
 		(at 142.24 133.35 0)
 		(unit 1)
@@
 			)
 		)
-		(property "ChipDip" ""
+		(property "ChipDip" "9020004445"
 			(at 142.24 133.35 0)
 			(effects
@@
 	)
 	(symbol
-		(lib_id "ProPrj_CAN-easyedapro:TJA1050DRG")
+		(lib_id "Local:TJA1050DRG")
 		(at 151.13 45.72 0)
 		(unit 1)
@@
 			)
 		)
-		(property "Footprint" "ProPrj_CAN_2025-04-09:SOIC-8E"
+		(property "Footprint" "Library:SOIC-8E"
 			(at 151.13 45.72 0)
 			(effects
@@
 			)
 		)
-		(property "ChipDip" ""
+		(property "ChipDip" "8044731834"
 			(at 151.13 45.72 0)
 			(effects
@@
 			)
 		)
-		(property "Value" "BOOT"
+		(property "Value" "PLS-3"
 			(at 221.488 70.104 0)
 			(effects
@@
 			)
 		)
-		(property "Datasheet" "~"
+		(property "Datasheet" "https://www.chipdip.ru/product/pls-3"
 			(at 217.17 69.85 0)
 			(effects
@@
 			)
 		)
-		(property "ChipDip" ""
+		(property "ChipDip" "132511368"
 			(at 217.17 69.85 0)
 			(effects
@@
 			)
 		)
-		(property "Datasheet" "~"
+		(property "Datasheet" "https://static.chipdip.ru/lib/295/DOC021295017.pdf"
 			(at 41.91 128.27 0)
 			(effects
@@
 			)
 		)
-		(property "ChipDip" ""
+		(property "ChipDip" "9001106124"
 			(at 41.91 128.27 0)
 			(effects
@@
 			)
 		)
-		(property "Datasheet" "~"
+		(property "Datasheet" "https://static.chipdip.ru/lib/175/DOC011175144.pdf"
 			(at 160.02 80.01 0)
 			(effects
@@
 			)
 		)
-		(property "ChipDip" ""
+		(property "ChipDip" "9000079736"
 			(at 160.02 80.01 0)
 			(effects
@@
 			)
 		)
-		(property "Footprint" "Diode_SMD:D_SMA"
+		(property "Footprint" "Diode_SMD:D_SMB-SMC_Universal_Handsoldering"
 			(at 27.94 137.16 0)
 			(effects
@@
 			)
 		)
-		(property "Datasheet" "https://www.littelfuse.com/media?resourcetype=datasheets&itemid=75e32973-b177-4ee3-a0ff-cedaf1abdb93&filename=smaj-datasheet"
+		(property "Datasheet" "https://www.chipdip.ru/product/smaj33ca-umw"
 			(at 22.86 137.16 0)
 			(effects
@@
 			)
 		)
-		(property "ChipDip" ""
+		(property "ChipDip" "9001169250"
 			(at 22.86 137.16 0)
 			(effects
@@
 			)
 		)
-		(property "Datasheet" "~"
+		(property "Datasheet" "https://www.chipdip.ru/product/grm188r72a104ka35d"
 			(at 49.53 139.7 0)
 			(effects
@@
 			)
 		)
-		(property "ChipDip" ""
+		(property "ChipDip" "9000121254"
 			(at 49.53 139.7 0)
 			(effects
@@
 	)
 	(symbol
-		(lib_id "Regulator_Switching:LM2575-5.0BT")
+		(lib_id "Local:LM2575-5.0BT")
 		(at 80.01 130.81 0)
 		(unit 1)
@@
 			)
 		)
-		(property "ChipDip" ""
+		(property "ChipDip" "9001087019"
 			(at 80.01 130.81 0)
 			(effects
@@
 			)
 		)
-		(property "Datasheet" "~"
+		(property "Datasheet" "https://static.chipdip.ru/lib/538/DOC012538954.pdf"
 			(at 67.31 101.6 0)
 			(effects
@@
 			)
 		)
-		(property "ChipDip" ""
+		(property "ChipDip" "183744283"
 			(at 67.31 101.6 0)
 			(effects
